File: WaveGenerator/midi/midi.kicad_pcb (KiCad board)
At the start: 2 copper layers, 16.3 x 20.1 mm, 5 parts, among them J1 MIDI IN, J2 Conn_01x04

Commit message: Wave gerber panelized
Routing:
- net GND: track 9.94 -> 34.7 mm
Other:
- board size 16.3 x 20.1 mm -> 16.3 x 20.4 mm
Changed lines of the file:
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@@
     (thickness 1.6)
     (drawings 4)
-    (tracks 23)
+    (tracks 35)
     (zones 0)
     (modules 5)
@@
     (add_net "Net-(J1-Pad4)")
   )
-  (module synth:MIDI_IN (layer B.Cu)
-    (at 115.316 85.598 270)
-    (fp_text reference J1 (at 0 3.31 270) (layer B.SilkS)
-      (effects (font (size 1 1) (thickness 0.15)) (justify mirror))
-    )
-    (fp_text value "MIDI IN" (at 0 4.31 270) (layer B.Fab)
-      (effects (font (size 1 1) (thickness 0.15)) (justify mirror))
-    )
-    (fp_line (start -10.16 2.286) (end 9.906 2.286) (layer B.SilkS) (width 0.15))
-    (fp_line (start 9.906 2.286) (end 9.906 -10.16) (layer B.SilkS) (width 0.15))
-    (fp_line (start 9.906 -10.16) (end -10.16 -10.16) (layer B.SilkS) (width 0.15))
-    (fp_line (start -10.16 -10.16) (end -10.16 2.286) (layer B.SilkS) (width 0.15))
-    (fp_line (start -10.16 -8.382) (end 9.906 -8.382) (layer B.SilkS) (width 0.15))
-    (pad 1 thru_hole circle (at 7.62 0 270) (size 1.524 1.524) (drill 0.762) (layers *.Cu *.Mask)
-      (net 4 "Net-(J1-Pad1)"))
-    (pad 2 thru_hole circle (at 0 0 270) (size 1.524 1.524) (drill 0.762) (layers *.Cu *.Mask)
-      (net 2 "Net-(C2-Pad2)"))
-    (pad 3 thru_hole circle (at -7.62 0 270) (size 1.524 1.524) (drill 0.762) (layers *.Cu *.Mask)
-      (net 5 "Net-(J1-Pad3)"))
-    (pad 4 thru_hole circle (at 5.08 2.286 270) (size 1.524 1.524) (drill 0.762) (layers *.Cu *.Mask)
-      (net 3 "Net-(J1-Pad4)"))
-    (pad 5 thru_hole circle (at -5.08 2.286 270) (size 1.524 1.524) (drill 0.762) (layers *.Cu *.Mask)
-      (net 7 D2))
-    (pad "" thru_hole circle (at -7.62 -5.08 270) (size 3 3) (drill 2.4) (layers *.Cu *.Mask))
-    (pad "" thru_hole circle (at 7.874 -5.08 270) (size 3 3) (drill 2.5) (layers *.Cu *.Mask))
-    (pad "" thru_hole circle (at 5.08 -10.16 270) (size 1.524 1.524) (drill 0.762) (layers *.Cu *.Mask))
-    (pad "" thru_hole circle (at -5.08 -10.16 270) (size 1.524 1.524) (drill 0.762) (layers *.Cu *.Mask))
-  )
   (module Diode_THT:D_DO-35_SOD27_P7.62mm_Horizontal (layer F.Cu)
     (at 119.126 81.788 270)
@@
     )
   )
-  (gr_line (start 125.476 95.758) (end 109.22 95.758) (layer Edge.Cuts) (width 0.15))
-  (gr_line (start 125.476 75.692) (end 125.476 95.758) (layer Edge.Cuts) (width 0.15))
-  (gr_line (start 109.22 75.692) (end 125.476 75.692) (layer Edge.Cuts) (width 0.15))
-  (gr_line (start 109.22 95.758) (end 109.22 75.692) (layer Edge.Cuts) (width 0.15))
+  (module synth:MIDI_IN (layer B.Cu)
+    (at 115.316 85.598 270)
+    (fp_text reference J1 (at 0 3.31 270) (layer B.SilkS)
+      (effects (font (size 1 1) (thickness 0.15)) (justify mirror))
+    )
+    (fp_text value "MIDI IN" (at 0 4.31 270) (layer B.Fab)
+      (effects (font (size 1 1) (thickness 0.15)) (justify mirror))
+    )
+    (fp_line (start -10.16 2.286) (end 10.16 2.286) (layer B.SilkS) (width 0.15))
+    (fp_line (start 10.16 2.286) (end 10.16 -10.16) (layer B.SilkS) (width 0.15))
+    (fp_line (start 10.16 -10.16) (end -10.16 -10.16) (layer B.SilkS) (width 0.15))
+    (fp_line (start -10.16 -10.16) (end -10.16 2.286) (layer B.SilkS) (width 0.15))
+    (fp_line (start -10.16 -8.382) (end 10.16 -8.382) (layer B.SilkS) (width 0.15))
+    (pad 1 thru_hole circle (at 7.62 0 270) (size 1.524 1.524) (drill 0.762) (layers *.Cu *.Mask)
+      (net 4 "Net-(J1-Pad1)"))
+    (pad 2 thru_hole circle (at 0 0 270) (size 1.524 1.524) (drill 0.762) (layers *.Cu *.Mask)
+      (net 2 "Net-(C2-Pad2)"))
+    (pad 3 thru_hole circle (at -7.62 0 270) (size 1.524 1.524) (drill 0.762) (layers *.Cu *.Mask)
+      (net 5 "Net-(J1-Pad3)"))
+    (pad 4 thru_hole circle (at 5.08 2.286 270) (size 1.524 1.524) (drill 0.762) (layers *.Cu *.Mask)
+      (net 3 "Net-(J1-Pad4)"))
+    (pad 5 thru_hole circle (at -5.08 2.286 270) (size 1.524 1.524) (drill 0.762) (layers *.Cu *.Mask)
+      (net 7 D2))
+    (pad "" thru_hole circle (at -7.62 -5.08 270) (size 3 3) (drill 2.4) (layers *.Cu *.Mask))
+    (pad "" thru_hole circle (at 7.874 -5.08 270) (size 3 3) (drill 2.5) (layers *.Cu *.Mask))
+    (pad "" thru_hole circle (at 5.08 -10.16 270) (size 1.524 1.524) (drill 0.762) (layers *.Cu *.Mask))
+    (pad "" thru_hole circle (at -5.08 -10.16 270) (size 1.524 1.524) (drill 0.762) (layers *.Cu *.Mask))
+  )
+  (gr_line (start 125.476 75.3745) (end 109.22 75.3745) (layer Edge.Cuts) (width 0.15))
+  (gr_line (start 125.476 95.8215) (end 125.476 75.3745) (layer Edge.Cuts) (width 0.15))
+  (gr_line (start 109.22 95.8215) (end 109.22 75.3745) (layer Edge.Cuts) (width 0.2))
+  (gr_line (start 125.476 95.8215) (end 109.22 95.8215) (layer Edge.Cuts) (width 0.15))
   (segment (start 112.014 83.312) (end 110.998 84.328) (width 0.25) (layer F.Cu) (net 1))
   (segment (start 113.741 83.312) (end 112.014 83.312) (width 0.25) (layer F.Cu) (net 1))
@@
   (segment (start 112.268 89.238) (end 112.098 89.408) (width 0.25) (layer B.Cu) (net 1))
   (segment (start 112.268 85.598) (end 112.268 89.238) (width 0.25) (layer B.Cu) (net 1))
+  (segment (start 110.998 89.408) (end 110.998 91.059) (width 0.25) (layer F.Cu) (net 1))
+  (segment (start 110.998 91.059) (end 112.014 92.075) (width 0.25) (layer F.Cu) (net 1))
+  (segment (start 112.014 92.075) (end 114.427 92.075) (width 0.25) (layer F.Cu) (net 1))
+  (segment (start 114.427 92.075) (end 115.189 91.313) (width 0.25) (layer F.Cu) (net 1))
+  (segment (start 115.189 91.313) (end 122.047 91.313) (width 0.25) (layer F.Cu) (net 1))
+  (segment (start 113.741 83.312) (end 113.741 82.728) (width 0.25) (layer F.Cu) (net 1))
+  (segment (start 113.741 82.728) (end 114.046 82.423) (width 0.25) (layer F.Cu) (net 1))
+  (segment (start 114.046 82.423) (end 115.951 82.423) (width 0.25) (layer F.Cu) (net 1))
+  (segment (start 115.951 82.423) (end 118.618 85.09) (width 0.25) (layer F.Cu) (net 1))
+  (segment (start 110.998 89.408) (end 111.887 89.408) (width 0.25) (layer F.Cu) (net 1))
+  (segment (start 111.887 89.408) (end 112.649 88.646) (width 0.25) (layer F.Cu) (net 1))
+  (segment (start 112.649 88.646) (end 115.316 88.646) (width 0.25) (layer F.Cu) (net 1))
   (segment (start 115.316 85.598) (end 115.316 83.312) (width 0.25) (layer F.Cu) (net 2))
   (segment (start 114.10763 90.678) (end 113.03 90.678) (width 0.25) (layer F.Cu) (net 3))
@@
     (polygon
       (pts
-        (xy 109.22 75.692) (xy 126.238 75.692) (xy 126.238 95.758) (xy 109.22 95.758)
+        (xy 108.712 74.422) (xy 126.111 74.168) (xy 126.365 96.901) (xy 108.331 96.901)
       )
     )
