File: VCO_Eurotrack/vco/vco.kicad_pcb (KiCad board)
At the start: 2 copper layers, 59.4 x 80 mm, 71 parts, among them J1 EXP_FM, J10 SAW, J11 Conn_02x05_Odd_Even, J2 LIN_FM, J3 PWM_IN, J4 CV 1V/OCT, J5 SYNC_IN, J6 SINE, J7 TRI, J8 SQUARE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

Commit message: VCO board
Routing:
- net GND: track 5.08 -> 170.2 mm, vias 0 -> 13
- net +12V: track 24.8 -> 130.9 mm, vias 0 -> 4
- net VFCI: track 30.6 -> 128.3 mm, vias 0 -> 2
- net -12V: track 5.33 -> 91.2 mm, vias 0 -> 2
- net Net-(C2-Pad2): track 0.00 -> 66.3 mm
- net Net-(C6-Pad2): track 2.40 -> 63.8 mm, vias 0 -> 2
- net VPWM: track 0.00 -> 56.1 mm, vias 0 -> 1
- net Net-(R21-Pad2): track 0.00 -> 53.5 mm, vias 0 -> 4
- net Net-(R28-Pad2): track 0.00 -> 51.4 mm, vias 0 -> 4
- net Net-(R17-Pad1): track 2.62 -> 53.7 mm
- net REE: track 3.32 -> 48.6 mm, vias 0 -> 2
- net Net-(R29-Pad2): track 0.00 -> 43.5 mm, vias 0 -> 2
- net TRI_OUT: track 8.09 -> 51.1 mm, vias 0 -> 2
- net Net-(Q1-Pad3): track 11.2 -> 53.4 mm, vias 0 -> 1
- net Net-(R11-Pad2): track 0.00 -> 40.6 mm, vias 0 -> 2
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Other:
- board size 59.4 x 80 mm -> 61 x 80 mm
