File: vca/vca.kicad_pcb (KiCad board)
At the start: 2 copper layers, 67.9 x 71.2 mm, 43 parts, among them J1 IN1, J2 VC1, J3 OUT1, J4 IN2, J5 VC2, J6 OUT2, J8 Conn_02x05_Odd_Even, Q1 2N3906, Q2 2N3906, U1 TL074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

Commit message: Modified the eurorackpin schematic and cleaned up
Connections:
- D4 pad 1: 12V_ -> /EURORACKPIN/12Vto5V
- D4 pad 2: GND -> 12VC
- D5 pad 1: GND -> -12VC
- D5 pad 2: -12V_ -> Net-(D5-Pad2)
- L1 pad 1: 12VC -> /EURORACKPIN/12Vto5V
- L2 pad 1: -12VC -> Net-(D5-Pad2)
Routing:
- net GND: track 74.7 -> 58.0 mm
- net -12VC: track 5.84 -> 22.0 mm
- net 12VC: track 5.84 -> 20.5 mm
- net Net-(D5-Pad2): track 0.00 -> 11.9 mm
- net /EURORACKPIN/12Vto5V: track 0.00 -> 11.1 mm
- net -12V_: track 159.9 -> 154.2 mm
- net 12V_: track 157.9 -> 156.0 mm
